File: stemcell.kicad_pcb (KiCad board)
At the start: 2 copper layers, 17.8 x 31.9 mm, 36 parts, among them J1 USB C Connector, J2 Left, J3 Right, J4 Down, SW1 Boot0, U1 STM32F4x1CxUx, U2 XC6220B331MR, Y1 HSE1 8Mhz 12pF

Commit message: silkscreen
Parts:
- removed the G*** at (93.3, 68.3)
