File: stemcell.kicad_sch (KiCad schematic)
At the start: 36 parts, among them J1 USB C Connector, J2 Left, J3 Right, J4 Down, SW1 Boot0, U1 STM32F4x1CxUx, U2 XC6220B331MR, Y1 HSE1 8Mhz 12pF

Commit message: remove castellated pads
Parts:
- J2, J3: footprint stemcell:Pins12_castellated -> stemcell:Pins12
- J4: footprint stemcell:Pins5_castellated -> stemcell:Pins5
Changed lines of the file:
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@@
       (effects (font (size 1.27 1.27)) (justify left))
     )
-    (property "Footprint" "stemcell:Pins12_castellated" (id 2) (at 198.501 45.9486 0)
+    (property "Footprint" "stemcell:Pins12" (id 2) (at 198.501 45.9486 0)
       (effects (font (size 1.27 1.27)) hide)
     )
@@
     (property "Reference" "J4" (id 0) (at 205.6638 70.358 90))
     (property "Value" "Down" (id 1) (at 205.6638 72.263 90))
-    (property "Footprint" "stemcell:Pins5_castellated" (id 2) (at 205.6384 75.6158 0)
+    (property "Footprint" "stemcell:Pins5" (id 2) (at 205.6384 75.6158 0)
       (effects (font (size 1.27 1.27)) hide)
     )
@@
       (effects (font (size 1.27 1.27)) (justify left))
     )
-    (property "Footprint" "stemcell:Pins12_castellated" (id 2) (at 211.201 45.9486 0)
+    (property "Footprint" "stemcell:Pins12" (id 2) (at 211.201 45.9486 0)
       (effects (font (size 1.27 1.27)) hide)
     )
@@
     )
     (path "/30cde441-a4b4-4a86-92b5-1140e5d06e66"
-      (reference "J2") (unit 1) (value "Left") (footprint "stemcell:Pins12_castellated")
+      (reference "J2") (unit 1) (value "Left") (footprint "stemcell:Pins12")
     )
     (path "/9d72ddaf-d37c-44f1-b2cb-b3c798045fcb"
-      (reference "J3") (unit 1) (value "Right") (footprint "stemcell:Pins12_castellated")
+      (reference "J3") (unit 1) (value "Right") (footprint "stemcell:Pins12")
     )
     (path "/41715acf-7b81-4792-bfde-7e1c2a5ef40d"
-      (reference "J4") (unit 1) (value "Down") (footprint "stemcell:Pins5_castellated")
+      (reference "J4") (unit 1) (value "Down") (footprint "stemcell:Pins5")
     )
     (path "/3b6d7996-cb03-421c-89b7-14690c1f4b89"

Commit message: change usb-c connector to part in stock at JLC
Parts:
- J1: LCSC C2681554 -> C963373
Changed lines of the file:
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@@
       (effects (font (size 1.27 1.27)) hide)
     )
-    (property "LCSC" "C2681554" (id 4) (at 123.952 54.229 0)
+    (property "LCSC" "C963373 " (id 4) (at 123.952 54.229 0)
       (effects (font (size 1.27 1.27)) hide)
     )
